Commit message: Arrumada o eixo das juntas das rodas e o ackermann_controller (Teleop funfando no robô)

File: Programação/RPi4/catkin_ws/src/ackermann_vehicle_description/robot/urdf/Ackermann_robot.urdf (robot description, URDF)
Before this commit: robot Ackermann_robot, 10 links, 9 joints
Links:
- link chassi_link: geometry collision box size=0.22043 0.27703 0.12452; visual mesh filename=package://ackermann_vehicle_description/robot/meshes/stl/Ba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 scale=1.0 1.0 1.0
- link link_acker_front_left: geometry visual mesh filename=package://ackermann_vehicle_description/robot/meshes/stl/en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 scale=1.0 1.0 1.0
- link link_acker_front_right: geometry visual mesh filename=package://ackermann_vehicle_description/robot/meshes/stl/en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 scale=1.0 1.0 1.0
- link link_wheel_front_left: geometry collision cylinder length=0.05 radius=0.05; visual mesh filename=package://ackermann_vehicle_description/robot/meshes/stl/wh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 scale=1.0 1.0 1.0
- link link_wheel_front_right: geometry collision cylinder length=0.05 radius=0.05; visual mesh filename=package://ackermann_vehicle_description/robot/meshes/stl/wh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 scale=1.0 1.0 1.0
- link link_wheel_rear_left: geometry collision cylinder length=0.05 radius=0.05; visual mesh filename=package://ackermann_vehicle_description/robot/meshes/stl/wh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 scale=1.0 1.0 1.0
- link link_wheel_rear_right: geometry collision cylinder length=0.05 radius=0.05; visual mesh filename=package://ackermann_vehicle_description/robot/meshes/stl/wh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 scale=1.0 1.0 1.0

File: Programação/RPi4/catkin_ws/src/ackermann_vehicle_description/robot/urdf/torno_arckermann_joints.xacro (robot description, xacro)
@@ -1,4 +1,6 @@
 <?xml version="1.0" encoding="utf-8"?>
 <robot xmlns:xacro="http://ros.org/wiki/xacro">
+    <xacro:property name="degrees_45" value="0.785398163"/>
+    <xacro:property name="degrees_90" value="1.57079633"/>
     <joint name="joint_acker_front_left" type="revolute">
       <origin xyz="0.10378 -0.21397 -0.0371" rpy="0 0 0"/>
@@ -6,5 +8,5 @@
       <child link="link_acker_front_left"/>
       <axis xyz="0 0 1.0"/>
-      <limit lower="-3.14" upper="3.14" effort="5.0" velocity="15.0"/>
+      <limit lower="-${degrees_45}" upper="${degrees_45}" effort="5.0" velocity="15.0"/>
     </joint>
     <joint name="joint_acker_front_right" type="revolute">
@@ -13,5 +15,5 @@
       <child link="link_acker_front_right"/>
       <axis xyz="0 0 1.0"/>
-      <limit lower="-3.14" upper="3.14" effort="5.0" velocity="15.0"/>
+      <limit lower="-${degrees_45}" upper="${degrees_45}" effort="5.0" velocity="15.0"/>
     </joint>
 </robot>

File: Programação/RPi4/catkin_ws/src/ackermann_vehicle_description/robot/urdf/wheels_joints.xacro (robot description, xacro)
@@ -1,35 +1,38 @@
 <?xml version="1.0" encoding="utf-8"?>
 <robot xmlns:xacro="http://ros.org/wiki/xacro">
-    <xacro:macro name="wheel_joint" params="preffix suffix">
-      <joint name="joint_wheel_${preffix}_${suffix}" type="continuous">
+    <xacro:macro name="wheel_joint_left" params="preffix">
+      <joint name="joint_wheel_${preffix}_left" type="continuous">
           <xacro:if value="${preffix == 'front'}">
-            <xacro:if value="${suffix == 'left'}">
-              <origin xyz="0.03048 0 0" rpy="0 1.5708 0"/>
-              <parent link="link_acker_front_left"/>
-            </xacro:if>
-            <xacro:unless value="${suffix == 'left'}">
-              <origin xyz="-0.03049 0 0" rpy="0 -1.5708 0"/>
-              <parent link="link_acker_front_right"/>
-            </xacro:unless>
+            <origin xyz="0.03048 0 0" rpy="0 1.5708 0"/>
+            <parent link="link_acker_front_left"/>
           </xacro:if>
           <xacro:unless value="${preffix == 'front'}">
-            <xacro:if value="${suffix == 'left'}">
-              <origin xyz="0.13691 0.00033 -0.0371" rpy="0 1.5708 0"/>
-              <parent link="base_link"/>
-            </xacro:if>
-            <xacro:unless value="${suffix == 'left'}">
-              <origin xyz="-0.13691 0.00033 -0.0371" rpy="0 -1.5708 0"/>
-              <parent link="base_link"/>
-            </xacro:unless>
+            <origin xyz="0.13691 0.00033 -0.0371" rpy="0 1.5708 0"/>
+            <parent link="base_link"/>
           </xacro:unless>
-        <child link="link_wheel_${preffix}_${suffix}"/>
+        <child link="link_wheel_${preffix}_left"/>
         <axis xyz="0 0 1.0"/>
         <limit effort="1.0" velocity="100.0"/>
       </joint>
     </xacro:macro>
-    <xacro:wheel_joint preffix="front" suffix="left"/>
-    <xacro:wheel_joint preffix="front" suffix="right"/>
-    <xacro:wheel_joint preffix="rear" suffix="left"/>
-    <xacro:wheel_joint preffix="rear" suffix="right"/>
+    <xacro:macro name="wheel_joint_right" params="preffix">
+      <joint name="joint_wheel_${preffix}_right" type="continuous">
+          <xacro:if value="${preffix == 'front'}">
+            <origin xyz="-0.03049 0 0" rpy="0 -1.5708 0"/>
+            <parent link="link_acker_front_right"/>
+          </xacro:if>
+          <xacro:unless value="${preffix == 'front'}">
+            <origin xyz="-0.13691 0.00033 -0.0371" rpy="0 -1.5708 0"/>
+            <parent link="base_link"/>
+          </xacro:unless>
+        <child link="link_wheel_${preffix}_right"/>
+        <axis xyz="0 0 -1.0"/>
+        <limit effort="1.0" velocity="100.0"/>
+      </joint>
+    </xacro:macro>
+    <xacro:wheel_joint_left preffix="front"/>
+    <xacro:wheel_joint_right preffix="front"/>
+    <xacro:wheel_joint_left preffix="rear"/>
+    <xacro:wheel_joint_right preffix="rear"/>
     <!--<joint name="joint_wheel_front_left" type="continuous">
       <origin xyz="0.03048 0 0" rpy="0 1.5708 0"/>
