Commit message: Teb adaptado para gerar trajetória a partir da posição do robô para um objetivo

File: Programação/RPi4/catkin_ws/src/ackermann_vehicle_description/robot/urdf/base.xacro (robot description, xacro)
@@ -38,5 +38,5 @@
     </joint>
     <joint name="base_link_front_joint" type="fixed">
-      <origin xyz="0 -0.21396 0" rpy="0 0 0"/>
+      <origin xyz="0 -0.21396 0" rpy="0 0 3.14159"/>
       <parent link="base_link"/>
       <child link="base_link_front"/>

Commit message: teste

File: Programação/RPi4/catkin_ws/src/ackermann_vehicle_description/robot/urdf/base.xacro (robot description, xacro)
@@ -9,5 +9,5 @@
       <color rgba="0.8 0.8 0.8 1.0"/>
     </material>
-    <link name="base_link"/>
+    <link name="base_link_rear"/>
     <link name="chassi_link">
       <inertial>
@@ -30,15 +30,15 @@
       </collision>
     </link>
-    <link name="base_link_front">
+    <link name="base_link">
     </link>
     <joint name="chassi_link_joint" type="fixed">
         <origin xyz="0 0 0" rpy="0 0 0"/>
-        <parent link="base_link" />
+        <parent link="base_link_rear" />
         <child link="chassi_link"/>
     </joint>
     <joint name="base_link_front_joint" type="fixed">
-      <origin xyz="0 -0.21396 0" rpy="0 0 3.14159"/>
-      <parent link="base_link"/>
-      <child link="base_link_front"/>
+      <origin xyz="0 -0.21396 0" rpy="0 0 -1.570795"/>
+      <parent link="base_link_rear"/>
+      <child link="base_link"/>
     </joint>
 </robot>

File: Programação/RPi4/catkin_ws/src/ackermann_vehicle_description/robot/urdf/imu.xacro (robot description, xacro)
@@ -26,5 +26,5 @@
     <joint name="imu_joint" type="fixed">
         <origin xyz="0 0 0.07077" rpy="0 0 0"/>
-        <parent link="base_link" />
+        <parent link="base_link_rear" />
         <child link="imu_link" />
     </joint>

File: Programação/RPi4/catkin_ws/src/ackermann_vehicle_description/robot/urdf/torno_arckermann_joints.xacro (robot description, xacro)
@@ -3,17 +3,18 @@
     <xacro:property name="degrees_45" value="0.785398163"/>
     <xacro:property name="degrees_90" value="1.57079633"/>
+    <xacro:property name="degrees_60" value="1.04719667"/>
     <joint name="joint_acker_front_left" type="revolute">
       <origin xyz="0.10378 -0.21397 -0.0371" rpy="0 0 0"/>
-      <parent link="base_link"/>
+      <parent link="base_link_rear"/>
       <child link="link_acker_front_left"/>
       <axis xyz="0 0 1.0"/>
-      <limit lower="-${degrees_45}" upper="${degrees_45}" effort="5.0" velocity="15.0"/>
+      <limit lower="-${degrees_60}" upper="${degrees_60}" effort="5.0" velocity="15.0"/>
     </joint>
     <joint name="joint_acker_front_right" type="revolute">
       <origin xyz="-0.10624 -0.21396 -0.0371" rpy="0 0 0"/>
-      <parent link="base_link"/>
+      <parent link="base_link_rear"/>
       <child link="link_acker_front_right"/>
       <axis xyz="0 0 1.0"/>
-      <limit lower="-${degrees_45}" upper="${degrees_45}" effort="5.0" velocity="15.0"/>
+      <limit lower="-${degrees_60}" upper="${degrees_60}" effort="5.0" velocity="15.0"/>
     </joint>
 </robot>

File: Programação/RPi4/catkin_ws/src/ackermann_vehicle_description/robot/urdf/wheels_joints.xacro (robot description, xacro)
@@ -9,5 +9,5 @@
           <xacro:unless value="${preffix == 'front'}">
             <origin xyz="0.13691 0.00033 -0.0371" rpy="0 1.5708 0"/>
-            <parent link="base_link"/>
+            <parent link="base_link_rear"/>
           </xacro:unless>
         <child link="link_wheel_${preffix}_left"/>
@@ -24,5 +24,5 @@
           <xacro:unless value="${preffix == 'front'}">
             <origin xyz="-0.13691 0.00033 -0.0371" rpy="0 -1.5708 0"/>
-            <parent link="base_link"/>
+            <parent link="base_link_rear"/>
           </xacro:unless>
         <child link="link_wheel_${preffix}_right"/>

Commit message: Adicionado mapa da competição

File: Programação/RPi4/catkin_ws/src/ackermann_vehicle_description/robot/urdf/base.xacro (robot description, xacro)
@@ -9,5 +9,5 @@
       <color rgba="0.8 0.8 0.8 1.0"/>
     </material>
-    <link name="base_link_rear"/>
+    <link name="base_link"/>
     <link name="chassi_link">
       <inertial>
@@ -30,15 +30,15 @@
       </collision>
     </link>
-    <link name="base_link">
+    <link name="base_link_front">
     </link>
     <joint name="chassi_link_joint" type="fixed">
         <origin xyz="0 0 0" rpy="0 0 0"/>
-        <parent link="base_link_rear" />
+        <parent link="base_link" />
         <child link="chassi_link"/>
     </joint>
     <joint name="base_link_front_joint" type="fixed">
-      <origin xyz="0 -0.21396 0" rpy="0 0 -1.570795"/>
-      <parent link="base_link_rear"/>
-      <child link="base_link"/>
+      <origin xyz="0 -0.21396 0" rpy="0 0 0"/>
+      <parent link="base_link"/>
+      <child link="base_link_front"/>
     </joint>
 </robot>

File: Programação/RPi4/catkin_ws/src/ackermann_vehicle_description/robot/urdf/imu.xacro (robot description, xacro)
@@ -26,5 +26,5 @@
     <joint name="imu_joint" type="fixed">
         <origin xyz="0 0 0.07077" rpy="0 0 0"/>
-        <parent link="base_link_rear" />
+        <parent link="base_link" />
         <child link="imu_link" />
     </joint>

File: Programação/RPi4/catkin_ws/src/ackermann_vehicle_description/robot/urdf/torno_arckermann_joints.xacro (robot description, xacro)
@@ -6,5 +6,5 @@
     <joint name="joint_acker_front_left" type="revolute">
       <origin xyz="0.10378 -0.21397 -0.0371" rpy="0 0 0"/>
-      <parent link="base_link_rear"/>
+      <parent link="base_link"/>
       <child link="link_acker_front_left"/>
       <axis xyz="0 0 1.0"/>
@@ -13,5 +13,5 @@
     <joint name="joint_acker_front_right" type="revolute">
       <origin xyz="-0.10624 -0.21396 -0.0371" rpy="0 0 0"/>
-      <parent link="base_link_rear"/>
+      <parent link="base_link"/>
       <child link="link_acker_front_right"/>
       <axis xyz="0 0 1.0"/>

File: Programação/RPi4/catkin_ws/src/ackermann_vehicle_description/robot/urdf/wheels_joints.xacro (robot description, xacro)
@@ -9,5 +9,5 @@
           <xacro:unless value="${preffix == 'front'}">
             <origin xyz="0.13691 0.00033 -0.0371" rpy="0 1.5708 0"/>
-            <parent link="base_link_rear"/>
+            <parent link="base_link"/>
           </xacro:unless>
         <child link="link_wheel_${preffix}_left"/>
@@ -24,5 +24,5 @@
           <xacro:unless value="${preffix == 'front'}">
             <origin xyz="-0.13691 0.00033 -0.0371" rpy="0 -1.5708 0"/>
-            <parent link="base_link_rear"/>
+            <parent link="base_link"/>
           </xacro:unless>
         <child link="link_wheel_${preffix}_right"/>

Commit message: Atualizado o tf_publisher

File: Programação/RPi4/catkin_ws/src/ackermann_vehicle_description/robot/urdf/base.xacro (robot description, xacro)
@@ -38,5 +38,5 @@
     </joint>
     <joint name="base_link_front_joint" type="fixed">
-      <origin xyz="0 -0.21396 0" rpy="0 0 0"/>
+      <origin xyz="0 -0.10698 0" rpy="0 0 -1.570795"/>
       <parent link="base_link"/>
       <child link="base_link_front"/>

Commit message: Arrumada orientação do base_link e de odom

File: Programação/RPi4/catkin_ws/src/ackermann_vehicle_description/robot/urdf/base.xacro (robot description, xacro)
@@ -33,5 +33,5 @@
     </link>
     <joint name="chassi_link_joint" type="fixed">
-        <origin xyz="0 0 0" rpy="0 0 0"/>
+        <origin xyz="0 0 0" rpy="0 0 3.141596"/>
         <parent link="base_link" />
         <child link="chassi_link"/>

File: Programação/RPi4/catkin_ws/src/ackermann_vehicle_description/robot/urdf/torno_arckermann_joints.xacro (robot description, xacro)
@@ -5,5 +5,5 @@
     <xacro:property name="degrees_60" value="1.04719667"/>
     <joint name="joint_acker_front_left" type="revolute">
-      <origin xyz="0.10378 -0.21397 -0.0371" rpy="0 0 0"/>
+      <origin xyz="0.10378 0.21397 -0.0371" rpy="0 0 0"/>
       <parent link="base_link"/>
       <child link="link_acker_front_left"/>
@@ -12,5 +12,5 @@
     </joint>
     <joint name="joint_acker_front_right" type="revolute">
-      <origin xyz="-0.10624 -0.21396 -0.0371" rpy="0 0 0"/>
+      <origin xyz="-0.10624 0.21396 -0.0371" rpy="0 0 0"/>
       <parent link="base_link"/>
       <child link="link_acker_front_right"/>

Commit message: upando novamente o codigo

File: Programação/RPi4/catkin_ws/src/ackermann_vehicle_description/robot/urdf/base.xacro (robot description, xacro)
@@ -17,5 +17,5 @@
       </inertial>
       <visual name="Base">
-        <origin xyz="-0.00055 -0.06897 0.06435" rpy="0 -3.14159 -0.00587"/>
+        <origin xyz="-0.00055 -0.06897 0.06435" rpy="0 -3.14159 -0.00587""/>
         <geometry>
           <mesh filename="${BASE}" scale="1.0 1.0 1.0"/>
